File: EagleCAD/SpeedDemon/Schematic.brd (EAGLE design)
At the start: 100 x 80 mm, 66 parts, among them Q1 DMC2700, U3 LM3676, U4 STM32F072-LQFP48, X1 32.768kHz

Commit message: board layout.. needs some work
Parts:
- added C19: 1uF, 0805_generics:C_0805
- added C20: 100nF, 0805_generics:C_0805
- moved U1A 167.0 mm to (123.1, 29.2), turned to 270 degrees
- moved C17 165.7 mm to (117.2, 29.3)
- moved SIGNAL_OP 153.6 mm to (123.1, 23.4)
- moved C8 128.2 mm to (61.7, 31.8)
- moved C13 123.7 mm to (67.0, 43.8), turned to 270 degrees
- moved X1 115.6 mm to (48.5, 44.0), turned to 90 degrees
- moved C12 111.4 mm to (61.7, 35.0)
- moved C7 109.6 mm to (66.0, 39.2), turned to 270 degrees
- moved JP5 109.0 mm to (73.1, 36.0), turned to 270 degrees
- moved R11 103.1 mm to (35.8, 56.4), turned to 180 degrees
- moved C3 101.7 mm to (33.1, 63.3)
- moved L1 100.4 mm to (37.6, 43.7), turned to 270 degrees
- moved TM1 96.3 mm to (31.5, 32.2), turned to 180 degrees
- moved R15 90.9 mm to (65.9, 35.0), turned to 90 degrees
- moved D1 90.7 mm to (35.1, 53.7), turned to 180 degrees
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Connections:
- net +3V3: now also C19.1, C20.1
- net GND: now also C19.2, C20.2, U3.P$1, U4.10, U4.11, U4.12, U4.2, U4.27, U4.28, U4.29, U4.30, U4.31, U4.32, U4.33, U4.38, U4.42, U4.44, U4.45, U4.46, U4.5, U4.6
Routing:
- net VBATT+_SW: track 0.00 -> 94.3 mm, vias 0 -> 4
- net VBATT+: track 0.00 -> 94.3 mm, vias 0 -> 2
- net +3V3: track 70.0 -> 148.3 mm, vias 0 -> 5
- net GND: track 1.72 -> 63.4 mm, vias 1 -> 8
- net +V+_CHG: track 0.00 -> 59.2 mm, vias 0 -> 4
- net PWR_SW: track 0.00 -> 29.1 mm, vias 0 -> 2
- net N$31: track 0.00 -> 24.7 mm
- net FL_SWDIO: track 0.00 -> 21.5 mm, vias 0 -> 2
- net N$1: track 0.00 -> 20.9 mm, vias 0 -> 2
- net SENSOR_SIG_OP: track 0.00 -> 18.1 mm
- net FL_RESET: track 0.00 -> 17.2 mm, vias 0 -> 2
- net N$28: track 0.00 -> 16.5 mm
- net Q1_D1: track 0.00 -> 13.5 mm
- net SW_RIGHT: track 14.7 -> 27.5 mm, vias 0 -> 1
- net SW_DOWN: track 13.4 -> 25.5 mm, vias 0 -> 1
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- added copper zone on layer 1, net GND
- added copper zone on layer 16, net GND
- removed copper zone on layer 1, net +3V3
Other:
- board size 100 x 80 mm -> 77.5 x 47.5 mm
- board text added: "DNP"
